File: Game-Boy-Zero-DMG-Controller-PCB.sch (KiCad schematic (older format))
At the start: 11 parts, among them P1 CONN_01X11, SW1 LEFT, SW10 A, SW2 UP, SW3 RIGHT, SW4 DOWN, SW5 SELECT, SW6 START, SW7 X, SW8 Y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

Commit message: All buttons wired. About to connect GND
Parts:
- renumbered SW4 to SW3, SW3 to SW4
Changed lines of the file:
@@
 LIBS:contrib
 LIBS:valves
-LIBS:test-cache
+LIBS:Game-Boy-Zero-DMG-Controller-PCB-cache
 EELAYER 25 0
 EELAYER END
@@
 $EndComp
 $Comp
-L SW_PUSH SW3
+L SW_PUSH SW4
 U 1 1 58614398
 P 1750 2700
-F 0 "SW3" H 1900 2810 50  0000 C CNN
+F 0 "SW4" H 1900 2810 50  0000 C CNN
 F 1 "RIGHT" H 1750 2620 50  0000 C CNN
 F 2 "GameBoy:GameBoy-DMG-BTN" H 1750 2700 50  0001 C CNN
@@
 $EndComp
 $Comp
-L SW_PUSH SW4
+L SW_PUSH SW3
 U 1 1 58614485
 P 1750 3100
-F 0 "SW4" H 1900 3210 50  0000 C CNN
+F 0 "SW3" H 1900 3210 50  0000 C CNN
 F 1 "DOWN" H 1750 3020 50  0000 C CNN
 F 2 "GameBoy:GameBoy-DMG-BTN" H 1750 3100 50  0001 C CNN
