File: Game-Boy-Zero-DMG-Controller-PCB.kicad_pcb (KiCad board)
At the start: 2 copper layers, 81.3 x 52.3 mm, 22 parts, among them P1 CONN_01X11, SW1 LEFT, SW10 A, SW2 UP, SW3 RIGHT, SW4 DOWN, SW5 SELECT, SW6 START, SW7 X, SW8 Y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

Commit message: All buttons wired. About to connect GND
Parts:
- SW3: value RIGHT -> DOWN
- SW4: value DOWN -> RIGHT
- SW6: footprint GameBoy:GameBoy-DMG-SEL2 -> GameBoy:GameBoy-DMG-START-SEL
- moved P1 3.30 mm to (149.1, 78.2)
Connections:
- SW3 pad 2: Net-(P1-Pad4) -> Net-(P1-Pad5)
- SW4 pad 2: Net-(P1-Pad5) -> Net-(P1-Pad4)
Routing:
- net Net-(P1-Pad11): track 5.20 -> 47.0 mm
- net Net-(P1-Pad7): track 24.0 -> 63.0 mm
- net Net-(P1-Pad6): track 24.2 -> 61.9 mm
- net Net-(P1-Pad4): track 5.35 -> 39.1 mm
- net Net-(P1-Pad2): track 5.20 -> 37.7 mm
- net Net-(P1-Pad10): track 5.20 -> 35.5 mm
- net Net-(P1-Pad8): track 5.20 -> 34.5 mm
- net Net-(P1-Pad3): track 5.20 -> 28.5 mm
- net Net-(P1-Pad5): track 5.35 -> 27.4 mm
- net Net-(P1-Pad9): track 5.20 -> 22.2 mm
- net GND: track 99.6 -> 111.1 mm

Commit message: Route GND
Routing:
- net GND: track 111.1 -> 334.2 mm, vias 0 -> 10
Changed lines of the file:
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@@
   (general
     (links 88)
-    (no_connects 10)
-    (area 126.924999 72.2046 209.051258 127.075001)
+    (no_connects 0)
+    (area 126.924999 74.600999 208.355001 127.075001)
     (thickness 1.6)
     (drawings 21)
-    (tracks 173)
+    (tracks 228)
     (zones 0)
     (modules 22)
@@
   (gr_line (start 148.59 127) (end 148.59 118.11) (angle 90) (layer Edge.Cuts) (width 0.15))
   (gr_line (start 148.59 127) (end 179.578 127) (angle 90) (layer Edge.Cuts) (width 0.15))
+  (segment (start 141.986 94.742) (end 141.986 80.518) (width 0.1524) (layer B.Cu) (net 1))
+  (segment (start 144.272 78.232) (end 149.098 78.232) (width 0.1524) (layer B.Cu) (net 1) (status 800000))
+  (segment (start 141.986 80.518) (end 144.272 78.232) (width 0.1524) (layer B.Cu) (net 1))
+  (segment (start 174.752 115.316) (end 176.784 115.316) (width 0.1524) (layer B.Cu) (net 1))
+  (segment (start 176.784 115.316) (end 185.674 106.426) (width 0.1524) (layer B.Cu) (net 1))
+  (segment (start 159.512 115.316) (end 162.052 117.856) (width 0.1524) (layer B.Cu) (net 1))
+  (via (at 162.052 117.856) (size 0.6858) (drill 0.3302) (layers F.Cu B.Cu) (net 1))
+  (segment (start 162.052 117.856) (end 159.575635 117.856) (width 0.1524) (layer F.Cu) (net 1))
+  (segment (start 177.292 117.856) (end 174.752 115.316) (width 0.1524) (layer B.Cu) (net 1))
+  (via (at 177.292 117.856) (size 0.6858) (drill 0.3302) (layers F.Cu B.Cu) (net 1))
+  (segment (start 174.815635 117.856) (end 177.292 117.856) (width 0.1524) (layer F.Cu) (net 1))
+  (segment (start 153.924 113.284) (end 145.796 113.284) (width 0.1524) (layer B.Cu) (net 1))
+  (segment (start 155.956 115.316) (end 153.924 113.284) (width 0.1524) (layer B.Cu) (net 1))
+  (segment (start 174.752 115.316) (end 159.512 115.316) (width 0.1524) (layer B.Cu) (net 1))
+  (segment (start 159.512 115.316) (end 155.956 115.316) (width 0.1524) (layer B.Cu) (net 1))
+  (segment (start 185.674 106.426) (end 181.356 102.108) (width 0.1524) (layer B.Cu) (net 1))
+  (segment (start 181.356 102.108) (end 181.356 97.028) (width 0.1524) (layer B.Cu) (net 1))
+  (segment (start 181.356 97.028) (end 179.324 94.996) (width 0.1524) (layer B.Cu) (net 1))
+  (segment (start 179.324 94.996) (end 179.324 91.44) (width 0.1524) (layer B.Cu) (net 1))
+  (segment (start 200.152 99.314) (end 193.04 106.426) (width 0.1524) (layer B.Cu) (net 1))
+  (segment (start 193.04 106.426) (end 185.674 106.426) (width 0.1524) (layer B.Cu) (net 1))
+  (via (at 185.674 106.426) (size 0.6858) (drill 0.3302) (layers F.Cu B.Cu) (net 1))
+  (segment (start 185.674 106.426) (end 185.674 104.902) (width 0.1524) (layer F.Cu) (net 1))
+  (segment (start 193.802 84.582) (end 200.152 90.932) (width 0.1524) (layer B.Cu) (net 1))
+  (via (at 200.152 99.314) (size 0.6858) (drill 0.3302) (layers F.Cu B.Cu) (net 1))
+  (segment (start 200.152 99.314) (end 200.152 98.044) (width 0.1524) (layer F.Cu) (net 1))
+  (segment (start 200.152 90.932) (end 200.152 99.314) (width 0.1524) (layer B.Cu) (net 1))
+  (segment (start 179.324 91.44) (end 186.182 84.582) (width 0.1524) (layer B.Cu) (net 1))
+  (segment (start 186.182 84.582) (end 193.802 84.582) (width 0.1524) (layer B.Cu) (net 1))
+  (via (at 179.324 91.44) (size 0.6858) (drill 0.3302) (layers F.Cu B.Cu) (net 1))
+  (segment (start 179.324 90.17) (end 179.324 91.44) (width 0.1524) (layer F.Cu) (net 1))
+  (via (at 193.802 84.582) (size 0.6858) (drill 0.3302) (layers F.Cu B.Cu) (net 1))
+  (segment (start 193.802 84.582) (end 193.802 83.312) (width 0.1524) (layer F.Cu) (net 1))
+  (segment (start 141.986 94.742) (end 146.558 94.742) (width 0.1524) (layer B.Cu) (net 1))
+  (segment (start 150.876 99.06) (end 150.876 104.14) (width 0.1524) (layer B.Cu) (net 1))
+  (segment (start 146.558 94.742) (end 150.876 99.06) (width 0.1524) (layer B.Cu) (net 1))
+  (segment (start 141.986 94.742) (end 137.414 94.742) (width 0.1524) (layer B.Cu) (net 1))
+  (segment (start 141.986 93.726) (end 141.986 94.742) (width 0.1524) (layer F.Cu) (net 1))
+  (via (at 141.986 94.742) (size 0.6858) (drill 0.3302) (layers F.Cu B.Cu) (net 1))
+  (segment (start 132.588 99.568) (end 132.588 104.14) (width 0.1524) (layer B.Cu) (net 1))
+  (segment (start 137.414 94.742) (end 132.588 99.568) (width 0.1524) (layer B.Cu) (net 1))
+  (segment (start 150.876 104.14) (end 150.876 108.204) (width 0.1524) (layer B.Cu) (net 1))
+  (segment (start 150.876 108.204) (end 145.796 113.284) (width 0.1524) (layer B.Cu) (net 1))
+  (segment (start 145.796 113.284) (end 141.986 113.284) (width 0.1524) (layer B.Cu) (net 1))
+  (via (at 150.876 104.14) (size 0.6858) (drill 0.3302) (layers F.Cu B.Cu) (net 1))
+  (segment (start 150.876 102.87) (end 150.876 104.14) (width 0.1524) (layer F.Cu) (net 1))
+  (segment (start 132.588 104.14) (end 132.588 108.712) (width 0.1524) (layer B.Cu) (net 1))
+  (segment (start 132.588 108.712) (end 137.16 113.284) (width 0.1524) (layer B.Cu) (net 1))
+  (segment (start 137.16 113.284) (end 141.986 113.284) (width 0.1524) (layer B.Cu) (net 1))
+  (via (at 132.588 104.14) (size 0.6858) (drill 0.3302) (layers F.Cu B.Cu) (net 1))
+  (segment (start 132.588 104.14) (end 132.588 102.87) (width 0.1524) (layer F.Cu) (net 1))
+  (segment (start 141.986 112.014) (end 141.986 113.284) (width 0.1524) (layer F.Cu) (net 1))
+  (via (at 141.986 113.284) (size 0.6858) (drill 0.3302) (layers F.Cu B.Cu) (net 1))
+  (segment (start 174.210443 118.461192) (end 174.815635 117.856) (width 0.1524) (layer F.Cu) (net 1))
+  (segment (start 158.970443 118.461192) (end 159.575635 117.856) (width 0.1524) (layer F.Cu) (net 1))
   (segment (start 131.064 102.87) (end 132.588 102.87) (width 0.1524) (layer F.Cu) (net 1))
   (segment (start 132.588 102.87) (end 134.112 102.87) (width 0.1524) (layer F.Cu) (net 1))
@@
   (segment (start 151.892 120.396) (end 154.178 119.126) (width 0.1524) (layer F.Cu) (net 6))
   (segment (start 151.19982 122.506323) (end 154.796962 123.640497) (width 0.1524) (layer F.Cu) (net 6))
-  (segment (start 164.338 78.232) (end 164.338 112.182465) (width 0.1524) (layer F.Cu) (net 7) (status 400000))
-  (segment (start 164.338 112.182465) (end 171.847038 119.691503) (width 0.1524) (layer F.Cu) (net 7) (status 800000))
+  (segment (start 164.338 78.232) (end 164.338 112.182465) (width 0.1524) (layer F.Cu) (net 7))
+  (segment (start 164.338 112.182465) (end 171.847038 119.691503) (width 0.1524) (layer F.Cu) (net 7))
   (segment (start 166.43982 122.506323) (end 167.132 120.396) (width 0.1524) (layer F.Cu) (net 7))
   (segment (start 170.18 118.872) (end 171.847038 119.691503) (width 0.1524) (layer F.Cu) (net 7))

Commit message: Sign my name so that everyone knows how legit I am
Other:
- board text added: "DMG+ Control Panel"
- board text added: "flyingtoaster0"
Changed lines of the file:
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@@
     (area 126.924999 74.600999 208.355001 127.075001)
     (thickness 1.6)
-    (drawings 21)
+    (drawings 23)
     (tracks 228)
     (zones 0)
@@
       (effects (font (size 1.27 1.27) (thickness 0.1016)))
     )
-    (fp_text value START (at 0 -4.572 27.5) (layer F.SilkS)
+    (fp_text value START (at 1.905 -4.572 27.5) (layer F.SilkS)
       (effects (font (thickness 0.15)))
     )
@@
       (net 1 GND))
   )
+  (gr_text "DMG+ Control Panel" (at 165.862 104.648) (layer F.SilkS)
+    (effects (font (size 1.27 1.27) (thickness 0.254)))
+  )
+  (gr_text flyingtoaster0 (at 134.62 76.708) (layer F.SilkS)
+    (effects (font (size 1.27 1.27) (thickness 0.254)))
+  )
   (gr_text A (at 174.498 80.01 90) (layer F.SilkS)
-    (effects (font (size 1.27 1.27) (thickness 0.254)) (justify right))
+    (effects (font (size 0.762 0.762) (thickness 0.1905)) (justify right))
   )
   (gr_text B (at 171.958 80.01 90) (layer F.SilkS)
-    (effects (font (size 1.27 1.27) (thickness 0.254)) (justify right))
+    (effects (font (size 0.762 0.762) (thickness 0.1905)) (justify right))
   )
   (gr_text Y (at 169.418 80.01 90) (layer F.SilkS)
-    (effects (font (size 1.27 1.27) (thickness 0.254)) (justify right))
+    (effects (font (size 0.762 0.762) (thickness 0.1905)) (justify right))
   )
   (gr_text X (at 166.878 80.01 90) (layer F.SilkS)
-    (effects (font (size 1.27 1.27) (thickness 0.254)) (justify right))
+    (effects (font (size 0.762 0.762) (thickness 0.1905)) (justify right))
   )
   (gr_text START (at 164.338 80.01 90) (layer F.SilkS)
-    (effects (font (size 1.27 1.27) (thickness 0.254)) (justify right))
+    (effects (font (size 0.762 0.762) (thickness 0.1905)) (justify right))
   )
   (gr_text SEL (at 161.798 80.01 90) (layer F.SilkS)
-    (effects (font (size 1.27 1.27) (thickness 0.254)) (justify right))
+    (effects (font (size 0.762 0.762) (thickness 0.1905)) (justify right))
   )
   (gr_text RIGHT (at 159.258 80.01 90) (layer F.SilkS)
-    (effects (font (size 1.27 1.27) (thickness 0.254)) (justify right))
+    (effects (font (size 0.762 0.762) (thickness 0.1905)) (justify right))
   )
   (gr_text DOWN (at 156.718 80.01 90) (layer F.SilkS)
-    (effects (font (size 1.27 1.27) (thickness 0.254)) (justify right))
+    (effects (font (size 0.762 0.762) (thickness 0.1905)) (justify right))
   )
   (gr_text LEFT (at 151.638 80.01 90) (layer F.SilkS)
-    (effects (font (size 1.27 1.27) (thickness 0.254)) (justify right))
+    (effects (font (size 0.762 0.762) (thickness 0.1905)) (justify right))
   )
   (gr_text UP (at 154.178 80.01 90) (layer F.SilkS)
-    (effects (font (size 1.27 1.27) (thickness 0.254)) (justify right))
+    (effects (font (size 0.762 0.762) (thickness 0.1905)) (justify right))
   )
   (gr_text GND (at 149.098 80.01 90) (layer F.SilkS)
-    (effects (font (size 1.27 1.27) (thickness 0.254)) (justify right))
+    (effects (font (size 0.762 0.762) (thickness 0.1905)) (justify right))
   )
   (gr_arc (start 192.278 127) (end 179.578 127) (angle 90) (layer Edge.Cuts) (width 0.15))
